File: Usborne_Robot.kicad_sch (KiCad schematic)
At the start: 46 parts, among them J1 C64, J2 BBC, J3 Motor Battery, J4 Relay Battery, J5 To Robot, K1 ARM, K2 GRIPPER, K3 LEFT, K4 RIGHT, K5 DIRECTION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

Commit message: Thicker traces for motor signals, wide footprints for transistors.
Parts:
- Q1, Q2, Q3, Q4, Q5, Q6: footprint Package_TO_SOT_THT:TO-92L_Inline -> Package_TO_SOT_THT:TO-92L_Inline_Wide
Changed lines of the file:
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@@
       (effects (font (size 1.27 1.27)) (justify left))
     )
-    (property "Footprint" "Package_TO_SOT_THT:TO-92L_Inline" (at 130.81 65.405 0)
+    (property "Footprint" "Package_TO_SOT_THT:TO-92L_Inline_Wide" (at 130.81 65.405 0)
       (effects (font (size 1.27 1.27)) hide)
     )
@@
       (effects (font (size 1.27 1.27)) (justify left))
     )
-    (property "Footprint" "Package_TO_SOT_THT:TO-92L_Inline" (at 202.565 65.405 0)
+    (property "Footprint" "Package_TO_SOT_THT:TO-92L_Inline_Wide" (at 202.565 65.405 0)
       (effects (font (size 1.27 1.27)) hide)
     )
@@
       (effects (font (size 1.27 1.27)) (justify left))
     )
-    (property "Footprint" "Package_TO_SOT_THT:TO-92L_Inline" (at 130.81 132.715 0)
+    (property "Footprint" "Package_TO_SOT_THT:TO-92L_Inline_Wide" (at 130.81 132.715 0)
       (effects (font (size 1.27 1.27)) hide)
     )
@@
       (effects (font (size 1.27 1.27)) (justify left))
     )
-    (property "Footprint" "Package_TO_SOT_THT:TO-92L_Inline" (at 202.565 132.715 0)
+    (property "Footprint" "Package_TO_SOT_THT:TO-92L_Inline_Wide" (at 202.565 132.715 0)
       (effects (font (size 1.27 1.27)) hide)
     )
@@
       (effects (font (size 1.27 1.27)) (justify left))
     )
-    (property "Footprint" "Package_TO_SOT_THT:TO-92L_Inline" (at 428.625 58.42 0)
+    (property "Footprint" "Package_TO_SOT_THT:TO-92L_Inline_Wide" (at 428.625 58.42 0)
       (effects (font (size 1.27 1.27)) hide)
     )
@@
       (effects (font (size 1.27 1.27)) (justify left))
     )
-    (property "Footprint" "Package_TO_SOT_THT:TO-92L_Inline" (at 288.925 106.68 0)
-      (effects (font (size 1.27 1.27)) hide)
-    )
+    (property "Footprint" "Package_TO_SOT_THT:TO-92L_Inline_Wide" (at 288.925 106.68 0)
+      (effects (font (size 1.27 1.27)) hide)
+    )
